Commit message: it work

File: src/rosbot1/description/lidar.xacro (robot description, xacro)
@@ -3,5 +3,5 @@
     <joint name="lidar_joint" type="fixed">
         <origin xyz="0 0 0.1" rpy="0 0 0" />
-        <parent link="robot_joint" />
+        <parent link="robot_link" />
         <child link="lidar_frame" />
     </joint>

File: src/rosbot1/description/robot.urdf.xacro (robot description, xacro)
@@ -1,4 +1,6 @@
 <?xml version="1.0"?>
 <robot name="rosbot1" xmlns:xacro="http://www.ros.org/wiki/xacro">
+    <xacro:include filename="materials.xacro" />
     <xacro:include filename="robot_core.xacro" />
+    <xacro:include filename="lidar.xacro" />
 </robot>

File: src/rosbot1/description/robot_core.xacro (robot description, xacro)
@@ -2,78 +2,45 @@
 <robot xmlns:xacro="http://ros.org/wiki/xacro" name="robot_core">
     <!-- Define the mecanum wheel -->
-    <xacro:macro name="mecanum_wheel" params="prefix">
-        <joint name="${prefix}_joint" type="continuous">
-            <origin xyz="0 0 0" rpy="0 0 0"/>
-            <parent link="${prefix}_base_link"/>
-            <child link="${prefix}_wheel_link"/>
-            <axis xyz="0 0 1"/>
-        </joint>
+    <xacro:macro name="mecanum_wheel" params="prefix origin">
         <link name="${prefix}_wheel_link">
             <visual>
-                <!-- Add visual properties for the wheel -->
+                <geometry>
+                    <cylinder radius="0.1" length="0.05" />
+                    <material name="white">
+                        <color rgba="1 1 1 1" />
+                    </material>
+                </geometry>
             </visual>
             <collision>
-                <!-- Add collision properties for the wheel -->
+                <geometry>
+                    <cylinder radius="0.1" length="0.05" />
+                </geometry>
             </collision>
             <inertial>
-                <!-- Add inertial properties for the wheel -->
+                <mass value="0.1" />
+                <inertia ixx="0.001" ixy="0" ixz="0" iyy="0.001" iyz="0" izz="0.001" />
             </inertial>
         </link>
+        <joint name="${prefix}_joint" type="continuous">
+            <origin xyz="${origin}" rpy="0 0 0" />
+            <parent link="robot_link" />
+            <child link="${prefix}_wheel_link" />
+            <axis xyz="0 0 1" />
+        </joint>
     </xacro:macro>
     <!-- Define the robot base -->
-    <link name="base_link">
-        <visual>
-            <!-- Add visual properties for the base -->
-        </visual>
-        <collision>
-            <!-- Add collision properties for the base -->
-        </collision>
-        <inertial>
-            <!-- Add inertial properties for the base -->
-        </inertial>
-    </link>
-    <!-- Add mecanum wheels -->
-    <xacro:mecanum_wheel prefix="front_left"/>
-    <xacro:mecanum_wheel prefix="front_right"/>
-    <xacro:mecanum_wheel prefix="rear_left"/>
-    <xacro:mecanum_wheel prefix="rear_right"/>
+    <link name="base_link"></link>
     <!-- Define the robot -->
-    <link name="robot_link">
-        <visual>
-            <!-- Add visual properties for the robot -->
-        </visual>
-        <collision>
-            <!-- Add collision properties for the robot -->
-        </collision>
-        <inertial>
-            <!-- Add inertial properties for the robot -->
-        </inertial>
-    </link>
-    <!-- Connect the wheels to the base -->
-    <joint name="front_left_joint" type="fixed">
-        <origin xyz="0.25 0.25 0" rpy="0 0 0"/>
-        <parent link="base_link"/>
-        <child link="front_left_base_link"/>
-    </joint>
-    <joint name="front_right_joint" type="fixed">
-        <origin xyz="0.25 -0.25 0" rpy="0 0 0"/>
-        <parent link="base_link"/>
-        <child link="front_right_base_link"/>
-    </joint>
-    <joint name="rear_left_joint" type="fixed">
-        <origin xyz="-0.25 0.25 0" rpy="0 0 0"/>
-        <parent link="base_link"/>
-        <child link="rear_left_base_link"/>
-    </joint>
-    <joint name="rear_right_joint" type="fixed">
-        <origin xyz="-0.25 -0.25 0" rpy="0 0 0"/>
-        <parent link="base_link"/>
-        <child link="rear_right_base_link"/>
-    </joint>
+    <link name="robot_link"></link>
     <!-- Connect the robot to the base -->
     <joint name="robot_joint" type="fixed">
-        <origin xyz="0 0 0" rpy="0 0 0"/>
-        <parent link="base_link"/>
-        <child link="robot_link"/>
+        <origin xyz="0 0 0" rpy="0 0 0" />
+        <parent link="base_link" />
+        <child link="robot_link" />
     </joint>
+    <!-- Add mecanum wheels -->
+    <xacro:mecanum_wheel prefix="front_left" origin="0.25 0.25 0" />
+    <xacro:mecanum_wheel prefix="front_right" origin="0.25 -0.25 0" />
+    <xacro:mecanum_wheel prefix="rear_left" origin="-0.25 0.25 0" />
+    <xacro:mecanum_wheel prefix="rear_right" origin="-0.25 -0.25 0" />
 </robot>

Commit message: fix: Lidar

File: src/rosbot1/description/lidar.xacro (robot description, xacro)
@@ -2,27 +2,16 @@
 <robot xmlns:xacro="http://www.ros.org/wiki/xacro">
     <joint name="lidar_joint" type="fixed">
-        <origin xyz="0 0 0.1" rpy="0 0 0" />
+        <origin xyz="0 0 0.05" rpy="0 0 0" />
         <parent link="robot_link" />
-        <child link="lidar_frame" />
+        <child link="ldlidar_link" />
     </joint>
-    <link name="lidar_frame">
+    <link name="ldlidar_link">
         <visual>
             <origin xyz="0 0 0" rpy="0 0 0" />
             <geometry>
-                <cylinder radius="0.05" length="0.1" />
+                <cylinder radius="0.025" length="0.05" />
             </geometry>
             <material name="black" />
         </visual>
-        <collision>
-            <origin xyz="0 0 0" rpy="0 0 0" />
-            <geometry>
-                <cylinder radius="0.05" length="0.1" />
-            </geometry>
-        </collision>
-        <inertial>
-            <origin xyz="0 0 0" rpy="0 0 0" />
-            <mass value="0.1" />
-            <inertia ixx="0.0001" ixy="0.0" ixz="0.0" iyy="0.0001" iyz="0.0" izz="0.0001" />
-        </inertial>
     </link>
 </robot>

File: src/rosbot1/description/robot.urdf.xacro (robot description, xacro)
@@ -3,4 +3,5 @@
     <xacro:include filename="materials.xacro" />
     <xacro:include filename="robot_core.xacro" />
+    <xacro:include filename="robot_wheels.xacro" />
     <xacro:include filename="lidar.xacro" />
 </robot>

File: src/rosbot1/description/robot_core.xacro (robot description, xacro)
@@ -1,36 +1,19 @@
 <?xml version="1.0"?>
-<robot xmlns:xacro="http://ros.org/wiki/xacro" name="robot_core">
-    <!-- Define the mecanum wheel -->
-    <xacro:macro name="mecanum_wheel" params="prefix origin">
-        <link name="${prefix}_wheel_link">
-            <visual>
-                <geometry>
-                    <cylinder radius="0.1" length="0.05" />
-                    <material name="white">
-                        <color rgba="1 1 1 1" />
-                    </material>
-                </geometry>
-            </visual>
-            <collision>
-                <geometry>
-                    <cylinder radius="0.1" length="0.05" />
-                </geometry>
-            </collision>
-            <inertial>
-                <mass value="0.1" />
-                <inertia ixx="0.001" ixy="0" ixz="0" iyy="0.001" iyz="0" izz="0.001" />
-            </inertial>
-        </link>
-        <joint name="${prefix}_joint" type="continuous">
-            <origin xyz="${origin}" rpy="0 0 0" />
-            <parent link="robot_link" />
-            <child link="${prefix}_wheel_link" />
-            <axis xyz="0 0 1" />
-        </joint>
-    </xacro:macro>
+<robot xmlns:xacro="http://ros.org/wiki/xacro">
+    <xacro:property name="chassis_length" value="0.15"/>
+    <xacro:property name="chassis_width" value="0.10"/>
+    <xacro:property name="chassis_height" value="0.04"/>
     <!-- Define the robot base -->
     <link name="base_link"></link>
     <!-- Define the robot -->
-    <link name="robot_link"></link>
+    <link name="robot_link">
+        <visual>
+            <origin xyz="0 0 0"/>
+            <geometry>
+                <box size="${chassis_length} ${chassis_width} ${chassis_height}"/>
+            </geometry>
+            <material name="orange"/>
+        </visual>
+    </link>
     <!-- Connect the robot to the base -->
     <joint name="robot_joint" type="fixed">
@@ -39,8 +22,3 @@
         <child link="robot_link" />
     </joint>
-    <!-- Add mecanum wheels -->
-    <xacro:mecanum_wheel prefix="front_left" origin="0.25 0.25 0" />
-    <xacro:mecanum_wheel prefix="front_right" origin="0.25 -0.25 0" />
-    <xacro:mecanum_wheel prefix="rear_left" origin="-0.25 0.25 0" />
-    <xacro:mecanum_wheel prefix="rear_right" origin="-0.25 -0.25 0" />
 </robot>
